File: FlightBit.kicad_sch (KiCad schematic)
At the start: 61 parts, among them J1 SBUS, J2 USB_C_Receptacle_USB2.0, J3 PPM, J4 OUT, J5 Conn_01x02, J6 Conn_01x02, Q1 1P, SW1 SW_Push, U1 STM32F103C8Tx, U2 MPU-6050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

Commit message: add debug connector
Parts:
- added J7: Conn_01x04, myCustomLibs:pad_01x04, symbol Connector_Generic:Conn_01x04
- NT1: footprint NetTie:NetTie-2_SMD_Pad0.5mm -> NetTie:NetTie-2_SMD_Pad2.0mm
Connections:
- net +3V3: now also J7.2 (Pin_2)
- net GND: now also J7.1 (Pin_1)
- net SWDIO: now reaches U1.34 (PA13)
- net SWDIO: now also J7.4 (Pin_4)
- net SWCLK: now reaches U1.37 (PA14)
- net SWCLK: now also J7.3 (Pin_3)
- no-connect marks 27 -> 25
Changed lines of the file:
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@@
   (no_connect (at 71.755 149.86))
   (no_connect (at 104.775 162.56))
-  (no_connect (at 104.775 160.02))
-  (no_connect (at 104.775 157.48))
   (no_connect (at 104.775 127))
   (no_connect (at 157.48 77.47))
@@
     (stroke (width 0) (type default) (color 0 0 0 0))
   )
+  (wire (pts (xy 104.775 160.02) (xy 111.125 160.02))
+    (stroke (width 0) (type default) (color 0 0 0 0))
+  )
   (wire (pts (xy 84.455 88.9) (xy 84.455 90.17))
     (stroke (width 0) (type default) (color 0 0 0 0))
@@
     (stroke (width 0) (type default) (color 0 0 0 0))
   )
+  (wire (pts (xy 109.22 78.105) (xy 111.125 78.105))
+    (stroke (width 0) (type default) (color 0 0 0 0))
+  )
+  (wire (pts (xy 104.775 157.48) (xy 111.125 157.48))
+    (stroke (width 0) (type default) (color 0 0 0 0))
+  )
   (wire (pts (xy 157.48 85.09) (xy 160.02 85.09))
     (stroke (width 0) (type default) (color 0 0 0 0))
@@
     (stroke (width 0) (type default) (color 0 0 0 0))
   )
+  (wire (pts (xy 109.22 80.645) (xy 111.125 80.645))
+    (stroke (width 0) (type default) (color 0 0 0 0))
+  )
   (wire (pts (xy 66.04 134.62) (xy 71.755 134.62))
     (stroke (width 0) (type default) (color 0 0 0 0))
@@
     (stroke (width 0) (type default) (color 0 0 0 0))
   )
+  (wire (pts (xy 109.22 75.565) (xy 111.125 75.565))
+    (stroke (width 0) (type default) (color 0 0 0 0))
+  )
+  (wire (pts (xy 109.22 83.185) (xy 111.125 83.185))
+    (stroke (width 0) (type default) (color 0 0 0 0))
+  )
   (polyline (pts (xy 128.27 13.97) (xy 180.975 13.97))
     (stroke (width 0) (type default) (color 0 0 0 0))
@@
     (effects (font (size 1.27 1.27)) (justify right bottom))
   )
+  (label "SWDIO" (at 111.125 157.48 0)
+    (effects (font (size 1.27 1.27)) (justify left bottom))
+  )
   (label "VBAT" (at 25.4 157.48 180)
     (effects (font (size 1.27 1.27)) (justify right bottom))
@@
     (effects (font (size 1.27 1.27)) (justify left bottom))
   )
+  (label "SWCLK" (at 111.125 160.02 0)
+    (effects (font (size 1.27 1.27)) (justify left bottom))
+  )
   (label "TIM3_S3" (at 199.39 96.52 0)
     (effects (font (size 1.27 1.27)) (justify left bottom))
@@
     (effects (font (size 1.27 1.27)) (justify left bottom))
   )
+  (label "SWDIO" (at 111.125 75.565 0)
+    (effects (font (size 1.27 1.27)) (justify left bottom))
+  )
   (label "USB_DN" (at 111.125 152.4 0)
     (effects (font (size 1.27 1.27)) (justify left bottom))
   )
+  (label "SWCLK" (at 111.125 78.105 0)
+    (effects (font (size 1.27 1.27)) (justify left bottom))
+  )
   (label "VBAT" (at 199.39 104.14 0)
     (effects (font (size 1.27 1.27)) (justify left bottom))
@@
     (pin "2")
   )
+  (symbol (lib_id "power:+3.3V") (at 111.125 80.645 270) (unit 1)
+    (in_bom yes) (on_board yes) (fields_autoplaced)
+    (property "Reference" "#PWR051" (id 0) (at 107.315 80.645 0)
+      (effects (font (size 1.27 1.27)) hide)
+    )
+    (property "Value" "+3.3V" (id 1) (at 114.3 80.6449 90)
+      (effects (font (size 1.27 1.27)) (justify left))
+    )
+    (property "Footprint" "" (id 2) (at 111.125 80.645 0)
+      (effects (font (size 1.27 1.27)) hide)
+    )
+    (property "Datasheet" "" (id 3) (at 111.125 80.645 0)
+      (effects (font (size 1.27 1.27)) hide)
+    )
+    (pin "1")
+  )
   (symbol (lib_id "power:GNDPWR") (at 244.475 155.575 0) (unit 1)
     (in_bom yes) (on_board yes) (fields_autoplaced)
@@
     (pin "1")
   )
+  (symbol (lib_id "Connector_Generic:Conn_01x04") (at 104.14 80.645 180) (unit 1)
+    (in_bom yes) (on_board yes) (fields_autoplaced)
+    (property "Reference" "J7" (id 0) (at 104.14 68.58 0))
+    (property "Value" "Conn_01x04" (id 1) (at 104.14 71.12 0))
+    (property "Footprint" "myCustomLibs:pad_01x04" (id 2) (at 104.14 80.645 0)
+      (effects (font (size 1.27 1.27)) hide)
+    )
+    (property "Datasheet" "~" (id 3) (at 104.14 80.645 0)
+      (effects (font (size 1.27 1.27)) hide)
+    )
+    (pin "1")
+    (pin "2")
+    (pin "3")
+    (pin "4")
+  )
   (symbol (lib_id "power:GND") (at 133.35 149.86 0) (unit 1)
     (in_bom yes) (on_board yes) (fields_autoplaced)
@@
     (property "Reference" "NT1" (id 0) (at 147.32 160.02 0))
     (property "Value" "NetTie_2" (id 1) (at 147.32 162.56 0))
-    (property "Footprint" "NetTie:NetTie-2_SMD_Pad0.5mm" (id 2) (at 147.32 165.735 0)
+    (property "Footprint" "NetTie:NetTie-2_SMD_Pad2.0mm" (id 2) (at 147.32 165.735 0)
       (effects (font (size 1.27 1.27)) hide)
     )
@@
     (pin "2")
   )
+  (symbol (lib_id "power:GND") (at 111.125 83.185 90) (unit 1)
+    (in_bom yes) (on_board yes) (fields_autoplaced)
+    (property "Reference" "#PWR052" (id 0) (at 117.475 83.185 0)
+      (effects (font (size 1.27 1.27)) hide)
+    )
+    (property "Value" "GND" (id 1) (at 114.935 83.1849 90)
+      (effects (font (size 1.27 1.27)) (justify right))
+    )
+    (property "Footprint" "" (id 2) (at 111.125 83.185 0)
+      (effects (font (size 1.27 1.27)) hide)
+    )
+    (property "Datasheet" "" (id 3) (at 111.125 83.185 0)
+      (effects (font (size 1.27 1.27)) hide)
+    )
+    (pin "1")
+  )
   (symbol (lib_id "Connector:USB_C_Receptacle_USB2.0") (at 142.24 87.63 0) (unit 1)
     (in_bom yes) (on_board yes) (fields_autoplaced)
@@
       (reference "#PWR050") (unit 1) (value "+5V") (footprint "")
     )
+    (path "/1648886e-dcab-42c9-a79b-cf14ab0627c2"
+      (reference "#PWR051") (unit 1) (value "+3.3V") (footprint "")
+    )
+    (path "/cfac05ee-a3ae-4795-8c87-951a67b2b9b0"
+      (reference "#PWR052") (unit 1) (value "GND") (footprint "")
+    )
     (path "/29956c9e-e58a-4fed-bce8-5cdcd2e07a06"
       (reference "C1") (unit 1) (value "100nF") (footprint "Capacitor_SMD:C_0402_1005Metric")
@@
       (reference "J6") (unit 1) (value "Conn_01x02") (footprint "myCustomLibs:pad_01x02")
     )
+    (path "/8c072932-9187-4fbd-b9d9-ecf7a7632879"
+      (reference "J7") (unit 1) (value "Conn_01x04") (footprint "myCustomLibs:pad_01x04")
+    )
     (path "/68e9654a-8bce-4572-ac86-456a1ae8670d"
       (reference "L1") (unit 1) (value "15uH/3A") (footprint "Inductor_SMD:L_Neosid_SM-PIC0602H")
     )
     (path "/a069d27d-579c-40e3-b155-2f6f2ef21fab"
-      (reference "NT1") (unit 1) (value "NetTie_2") (footprint "NetTie:NetTie-2_SMD_Pad0.5mm")
+      (reference "NT1") (unit 1) (value "NetTie_2") (footprint "NetTie:NetTie-2_SMD_Pad2.0mm")
     )
     (path "/c3ed69e3-6fec-4189-ba1c-1290aa00446d"
